Commit message: naming convention fixed

File: src/piper_ros/src/piper_moveit/piper_x_moveit/config/piper_x.ros2_control.xacro (robot description, xacro)
@@ -1,5 +1,5 @@
 <?xml version="1.0"?>
 <robot xmlns:xacro="http://www.ros.org/wiki/xacro">
-    <xacro:macro name="piper_ros2_control" params="name initial_positions_file">
+    <xacro:macro name="piper_x_ros2_control" params="name initial_positions_file">
         <xacro:property name="initial_positions" value="${load_yaml(initial_positions_file)['initial_positions']}"/>
         <ros2_control name="${name}" type="system">

File: src/piper_ros/src/piper_moveit/piper_x_moveit/config/piper_x.urdf.xacro (robot description, xacro)
@@ -1,9 +1,9 @@
 <?xml version="1.0"?>
-<robot xmlns:xacro="http://www.ros.org/wiki/xacro" name="piper">
+<robot xmlns:xacro="http://www.ros.org/wiki/xacro" name="piper_x">
     <xacro:arg name="initial_positions_file" default="initial_positions.yaml" />
     <!-- Import piper urdf file -->
     <xacro:include filename="$(find piper_x_description)/urdf/piper_x_description.xacro" />
     <!-- Import control_xacro -->
-    <xacro:include filename="piper.ros2_control.xacro" />
+    <xacro:include filename="piper_x.ros2_control.xacro" />
     <xacro:piper_ros2_control name="FakeSystem" initial_positions_file="$(arg initial_positions_file)"/>
 </robot>
