Commit message: moveit working with piperx

File: src/piper_ros/src/piper_description/piper_x_description/urdf/piper_x_description.xacro (robot description, xacro)
@@ -4,5 +4,11 @@
      For more information, please see http://wiki.ros.org/sw_urdf_exporter -->
 <robot xmlns:xacro="http://www.ros.org/wiki/xacro" name="piper_x_camera">
-<xacro:include filename="$(find realsense2_description)/urdf/test_d435_camera.urdf.xacro" />
+  <link name="world"/>
+  <joint name="world_to_base" type="fixed">
+    <parent link="world"/>
+    <child link="base_link"/>
+    <origin xyz="0 0 0" rpy="0 0 0"/>
+  </joint>
+<!-- <xacro:include filename="$(find realsense2_description)/urdf/test_d435_camera.urdf.xacro" /> -->
   <link
     name="base_link">
@@ -488,5 +494,5 @@
         <limit lower="-0.05" upper="0" effort="100" velocity="1" />
     </joint>
-    <link name="camera_stand_link">
+    <!-- <link name="camera_stand_link">
         <inertial>
             <origin xyz="0.0 0.0 0.0" rpy="0.0 0.0 0.0"/>
@@ -506,6 +512,6 @@
             </geometry>
         </collision>
-    </link>
-    <joint name="camera_stand_joint" type="fixed">
+    </link> -->
+    <!-- <joint name="camera_stand_joint" type="fixed">
         <origin xyz="0.001 -0.036 0.022" rpy="1.57 3.14 0.0"/>
         <parent link="link6"/>
@@ -520,4 +526,4 @@
         <axis xyz="0.0 0.0 0.0"/>
         <limit lower="0.0" upper="0.0" effort="0.0" velocity="0.0"/>
-    </joint>
+    </joint> -->
 </robot>

File: src/piper_ros/src/piper_description/piper_x_description/urdf/piper_x_description_d435.urdf (robot description, URDF)
Before this commit: robot piper_x_camera, 14 links, 13 joints
Links:
- removed link camera_stand_link

File: src/piper_ros/src/piper_moveit/piper_x_moveit/config/piper.urdf.xacro (robot description, xacro)
@@ -3,5 +3,5 @@
     <xacro:arg name="initial_positions_file" default="initial_positions.yaml" />
     <!-- Import piper urdf file -->
-    <xacro:include filename="$(find piper_description)/urdf/piper_description.xacro" />
+    <xacro:include filename="$(find piper_x_description)/urdf/piper_x_description.xacro" />
     <!-- Import control_xacro -->
     <xacro:include filename="piper.ros2_control.xacro" />

Commit message: fully working custom piper_x package (the one named custom not working)

File: src/piper_ros/src/piper_description/piper_x_description/urdf/piper_x_description.xacro (robot description, xacro)
@@ -4,10 +4,10 @@
      For more information, please see http://wiki.ros.org/sw_urdf_exporter -->
 <robot xmlns:xacro="http://www.ros.org/wiki/xacro" name="piper_x_camera">
-  <link name="world"/>
+  <!-- <link name="world"/>
   <joint name="world_to_base" type="fixed">
     <parent link="world"/>
     <child link="base_link"/>
     <origin xyz="0 0 0" rpy="0 0 0"/>
-  </joint>
+  </joint> -->
 <!-- <xacro:include filename="$(find realsense2_description)/urdf/test_d435_camera.urdf.xacro" /> -->
   <link
@@ -369,6 +369,6 @@
       xyz="0 0 1" />
     <limit
-      lower="-3.14"
-      upper="3.14"
+      lower="-1.57"
+      upper="1.57"
       effort="100"
       velocity="10" />

File: src/piper_ros/src/piper_moveit/piper_x_moveit_custom/config/piper_x_camera.ros2_control.xacro (robot description, xacro)
@@ -1,5 +1,5 @@
 <?xml version="1.0"?>
 <robot xmlns:xacro="http://www.ros.org/wiki/xacro">
-    <xacro:macro name="piper_ros2_control" params="name initial_positions_file">
+    <xacro:macro name="piper_x_camera_ros2_control" params="name initial_positions_file">
         <xacro:property name="initial_positions" value="${load_yaml(initial_positions_file)['initial_positions']}"/>
         <ros2_control name="${name}" type="system">

Commit message: fully working piper_x rviz moveit

File: src/piper_ros/src/piper_description/piper_x_description/urdf/piper_x_description.xacro (robot description, xacro)
@@ -3,11 +3,12 @@
      Commit Version: 1.6.0-4-g7f85cfe  Build Version: 1.6.7995.38578
      For more information, please see http://wiki.ros.org/sw_urdf_exporter -->
-<robot xmlns:xacro="http://www.ros.org/wiki/xacro" name="piper_x_camera">
-  <!-- <link name="world"/>
-  <joint name="world_to_base" type="fixed">
-    <parent link="world"/>
-    <child link="base_link"/>
-    <origin xyz="0 0 0" rpy="0 0 0"/>
-  </joint> -->
+<robot xmlns:xacro="http://www.ros.org/wiki/xacro" name="piper_x">
+  <!-- world -->
+  <link name="world"/>
+  <joint name="fixed_base_joint" type="fixed">
+      <parent link="world"/>
+      <child link="base_link"/>
+  </joint>
+<!-- arm -->
 <!-- <xacro:include filename="$(find realsense2_description)/urdf/test_d435_camera.urdf.xacro" /> -->
   <link
@@ -527,3 +528,24 @@
         <limit lower="0.0" upper="0.0" effort="0.0" velocity="0.0"/>
     </joint> -->
+  <!-- controller -->
+  <xacro:macro name="transmission_block" params="tran_name joint_name motor_name">
+    <transmission name="${tran_name}">
+        <type>transmission_interface/SimpleTransmission</type>
+        <joint name="${joint_name}">
+            <hardwareInterface>hardware_interface/PositionJointInterface</hardwareInterface>
+        </joint>
+        <actuator name="$motor_name">
+            <hardwareInterface>hardware_interface/PositionJointInterface</hardwareInterface>
+            <mechanicalReduction>1</mechanicalReduction>
+        </actuator>
+    </transmission>
+  </xacro:macro>
+  <xacro:transmission_block tran_name="tran1" joint_name="joint1" motor_name="motor1"/>
+  <xacro:transmission_block tran_name="tran2" joint_name="joint2" motor_name="motor2"/>
+  <xacro:transmission_block tran_name="tran3" joint_name="joint3" motor_name="motor3"/>
+  <xacro:transmission_block tran_name="tran4" joint_name="joint4" motor_name="motor4"/>
+  <xacro:transmission_block tran_name="tran5" joint_name="joint5" motor_name="motor5"/>
+  <xacro:transmission_block tran_name="tran6" joint_name="joint6" motor_name="motor6"/>
+  <xacro:transmission_block tran_name="tran7" joint_name="joint7" motor_name="motor7"/>
+  <xacro:transmission_block tran_name="tran8" joint_name="joint8" motor_name="motor8"/>
 </robot>

File: src/piper_ros/src/piper_moveit/piper_x_moveit/config/piper_x.urdf.xacro (robot description, xacro)
@@ -6,4 +6,4 @@
     <!-- Import control_xacro -->
     <xacro:include filename="piper_x.ros2_control.xacro" />
-    <xacro:piper_ros2_control name="FakeSystem" initial_positions_file="$(arg initial_positions_file)"/>
+    <xacro:piper_x_ros2_control name="FakeSystem" initial_positions_file="$(arg initial_positions_file)"/>
 </robot>
